Commit message: feat(sim): add gz ros2_control support for omni infantry

File: rmgo_ws/src/rmgo_description/urdf/omni_infantry.urdf.xacro (robot description, xacro)
@@ -4,4 +4,5 @@
   <xacro:property name="wheel_distance_y" value="0.31794"/>
   <xacro:property name="gimbal_center_height" value="0.32059"/>
+  <xacro:property name="controllers_file" value="$(find rmgo_description)/config/omni_infantry_controllers.yaml"/>
   <material name="white">
     <color rgba="1 1 1 1"/>
@@ -24,4 +25,5 @@
     <joint name="${name}_wheel_joint" type="continuous">
       <axis xyz="1 0 0"/>
+      <limit effort="20.0" velocity="40.0"/>
       <parent link="base_link"/>
       <child link="${name}_wheel_link"/>
@@ -50,4 +52,5 @@
   <joint name="yaw_joint" type="continuous">
     <axis xyz="0 0 1"/>
+    <limit effort="10.0" velocity="6.0"/>
     <parent link="base_link"/>
     <child link="yaw_link"/>
@@ -59,4 +62,5 @@
   <joint name="pitch_joint" type="continuous">
     <axis xyz="0 1 0"/>
+    <limit effort="10.0" velocity="6.0"/>
     <parent link="yaw_link"/>
     <child link="pitch_link"/>
@@ -80,3 +84,43 @@
     <origin xyz="0.06603 0 0.082"/>
   </joint>
+  <ros2_control name="OmniInfantryGz" type="system">
+    <hardware>
+      <plugin>gz_ros2_control/GazeboSimSystem</plugin>
+    </hardware>
+    <joint name="left_front_wheel_joint">
+      <command_interface name="velocity"/>
+      <state_interface name="position"/>
+      <state_interface name="velocity"/>
+    </joint>
+    <joint name="left_back_wheel_joint">
+      <command_interface name="velocity"/>
+      <state_interface name="position"/>
+      <state_interface name="velocity"/>
+    </joint>
+    <joint name="right_back_wheel_joint">
+      <command_interface name="velocity"/>
+      <state_interface name="position"/>
+      <state_interface name="velocity"/>
+    </joint>
+    <joint name="right_front_wheel_joint">
+      <command_interface name="velocity"/>
+      <state_interface name="position"/>
+      <state_interface name="velocity"/>
+    </joint>
+    <joint name="yaw_joint">
+      <command_interface name="position"/>
+      <state_interface name="position"/>
+      <state_interface name="velocity"/>
+    </joint>
+    <joint name="pitch_joint">
+      <command_interface name="position"/>
+      <state_interface name="position"/>
+      <state_interface name="velocity"/>
+    </joint>
+  </ros2_control>
+  <gazebo>
+    <plugin filename="libgz_ros2_control-system.so" name="gz_ros2_control::GazeboSimROS2ControlPlugin">
+      <parameters>${controllers_file}</parameters>
+    </plugin>
+  </gazebo>
 </robot>

Commit message: feat: add command bus and shooting chain

File: rmgo_ws/src/rmgo_description/urdf/omni_infantry.urdf.xacro (robot description, xacro)
@@ -2,4 +2,5 @@
 <robot name="omni_infantry" xmlns:xacro="http://www.ros.org/wiki/xacro">
   <xacro:arg name="hardware_plugin" default="rmgo_core/OmniInfantryGzInterface"/>
+  <xacro:arg name="command_hardware_plugin" default="rmgo_core/CommandGzInterface"/>
   <xacro:arg name="controllers_file" default="$(find rmgo_description)/config/omni_infantry_controllers.yaml"/>
   <xacro:property name="wheel_distance_x" value="0.31794"/>
@@ -8,4 +9,7 @@
   <material name="white">
     <color rgba="1 1 1 1"/>
+  </material>
+  <material name="black">
+    <color rgba="0.02 0.02 0.02 1"/>
   </material>
   <xacro:macro name="box_inertial" params="mass x y z">
@@ -117,4 +121,55 @@
     <child link="pitch_link"/>
   </joint>
+  <link name="left_friction_link">
+    <xacro:x_cylinder_inertial mass="0.08" radius="0.025" length="0.025"/>
+    <visual>
+      <origin rpy="0 ${pi/2} 0"/>
+      <geometry>
+        <cylinder radius="0.025" length="0.025"/>
+      </geometry>
+      <material name="black"/>
+    </visual>
+  </link>
+  <joint name="left_friction_joint" type="continuous">
+    <axis xyz="1 0 0"/>
+    <limit effort="2.0" velocity="800.0"/>
+    <parent link="pitch_link"/>
+    <child link="left_friction_link"/>
+    <origin xyz="0.075 0.04 0"/>
+  </joint>
+  <link name="right_friction_link">
+    <xacro:x_cylinder_inertial mass="0.08" radius="0.025" length="0.025"/>
+    <visual>
+      <origin rpy="0 ${pi/2} 0"/>
+      <geometry>
+        <cylinder radius="0.025" length="0.025"/>
+      </geometry>
+      <material name="black"/>
+    </visual>
+  </link>
+  <joint name="right_friction_joint" type="continuous">
+    <axis xyz="1 0 0"/>
+    <limit effort="2.0" velocity="800.0"/>
+    <parent link="pitch_link"/>
+    <child link="right_friction_link"/>
+    <origin xyz="0.075 -0.04 0"/>
+  </joint>
+  <link name="bullet_feeder_link">
+    <xacro:x_cylinder_inertial mass="0.12" radius="0.03" length="0.025"/>
+    <visual>
+      <origin rpy="0 ${pi/2} 0"/>
+      <geometry>
+        <cylinder radius="0.03" length="0.025"/>
+      </geometry>
+      <material name="white"/>
+    </visual>
+  </link>
+  <joint name="bullet_feeder_joint" type="continuous">
+    <axis xyz="1 0 0"/>
+    <limit effort="4.0" velocity="60.0"/>
+    <parent link="pitch_link"/>
+    <child link="bullet_feeder_link"/>
+    <origin xyz="-0.025 0 -0.035"/>
+  </joint>
   <link name="imu_link">
     <xacro:tiny_inertial mass="0.01"/>
@@ -175,4 +230,61 @@
       <state_interface name="velocity"/>
     </joint>
+    <joint name="left_friction_joint">
+      <command_interface name="velocity"/>
+      <command_interface name="effort"/>
+      <state_interface name="position"/>
+      <state_interface name="velocity"/>
+    </joint>
+    <joint name="right_friction_joint">
+      <command_interface name="velocity"/>
+      <command_interface name="effort"/>
+      <state_interface name="position"/>
+      <state_interface name="velocity"/>
+    </joint>
+    <joint name="bullet_feeder_joint">
+      <command_interface name="velocity"/>
+      <command_interface name="effort"/>
+      <state_interface name="position"/>
+      <state_interface name="velocity"/>
+    </joint>
+  </ros2_control>
+  <ros2_control name="CommandGz" type="system">
+    <hardware>
+      <plugin>$(arg command_hardware_plugin)</plugin>
+    </hardware>
+    <gpio name="command/chassis/linear/x">
+      <command_interface name="velocity"/>
+      <state_interface name="velocity"/>
+    </gpio>
+    <gpio name="command/chassis/linear/y">
+      <command_interface name="velocity"/>
+      <state_interface name="velocity"/>
+    </gpio>
+    <gpio name="command/chassis/angular/z">
+      <command_interface name="velocity"/>
+      <state_interface name="velocity"/>
+    </gpio>
+    <gpio name="command/chassis">
+      <command_interface name="mode"/>
+      <state_interface name="mode"/>
+    </gpio>
+    <gpio name="command/gimbal/yaw">
+      <command_interface name="velocity"/>
+      <state_interface name="velocity"/>
+    </gpio>
+    <gpio name="command/gimbal/pitch">
+      <command_interface name="velocity"/>
+      <state_interface name="velocity"/>
+    </gpio>
+    <gpio name="command/gimbal">
+      <command_interface name="enabled"/>
+      <state_interface name="enabled"/>
+    </gpio>
+    <gpio name="command/shooter">
+      <command_interface name="mode"/>
+      <command_interface name="sequence"/>
+      <state_interface name="mode"/>
+      <state_interface name="sequence"/>
+    </gpio>
   </ros2_control>
   <gazebo>

File: rmgo_ws/src/rmgo_description/urdf/omni_infantry_gz.urdf.xacro (robot description, xacro)
@@ -2,4 +2,5 @@
 <robot name="omni_infantry" xmlns:xacro="http://www.ros.org/wiki/xacro">
   <xacro:arg name="hardware_plugin" default="rmgo_core/OmniInfantryGzInterface"/>
+  <xacro:arg name="command_hardware_plugin" default="rmgo_core/CommandGzInterface"/>
   <xacro:arg name="controllers_file" default="$(find rmgo_description)/config/omni_infantry_controllers.yaml"/>
   <xacro:arg name="debug_visuals" default="false"/>
@@ -227,4 +228,40 @@
     <child link="pitch_link"/>
   </joint>
+  <link name="left_friction_link">
+    <xacro:x_cylinder_inertial mass="0.08" radius="0.025" length="0.025"/>
+    <xacro:debug_x_cylinder_visual name="left_friction_debug_visual" radius="0.025" length="0.025" material="black"/>
+  </link>
+  <joint name="left_friction_joint" type="continuous">
+    <axis xyz="1 0 0"/>
+    <limit effort="2.0" velocity="800.0"/>
+    <dynamics damping="0.0" friction="0.001"/>
+    <parent link="pitch_link"/>
+    <child link="left_friction_link"/>
+    <origin xyz="0.075 0.04 0"/>
+  </joint>
+  <link name="right_friction_link">
+    <xacro:x_cylinder_inertial mass="0.08" radius="0.025" length="0.025"/>
+    <xacro:debug_x_cylinder_visual name="right_friction_debug_visual" radius="0.025" length="0.025" material="black"/>
+  </link>
+  <joint name="right_friction_joint" type="continuous">
+    <axis xyz="1 0 0"/>
+    <limit effort="2.0" velocity="800.0"/>
+    <dynamics damping="0.0" friction="0.001"/>
+    <parent link="pitch_link"/>
+    <child link="right_friction_link"/>
+    <origin xyz="0.075 -0.04 0"/>
+  </joint>
+  <link name="bullet_feeder_link">
+    <xacro:x_cylinder_inertial mass="0.12" radius="0.03" length="0.025"/>
+    <xacro:debug_x_cylinder_visual name="bullet_feeder_debug_visual" radius="0.03" length="0.025" material="gimbal_orange"/>
+  </link>
+  <joint name="bullet_feeder_joint" type="continuous">
+    <axis xyz="1 0 0"/>
+    <limit effort="4.0" velocity="60.0"/>
+    <dynamics damping="0.01" friction="0.002"/>
+    <parent link="pitch_link"/>
+    <child link="bullet_feeder_link"/>
+    <origin xyz="-0.025 0 -0.035"/>
+  </joint>
   <link name="imu_link">
     <xacro:tiny_inertial mass="0.01"/>
@@ -299,4 +336,61 @@
       <state_interface name="velocity"/>
     </joint>
+    <joint name="left_friction_joint">
+      <command_interface name="velocity"/>
+      <command_interface name="effort"/>
+      <state_interface name="position"/>
+      <state_interface name="velocity"/>
+    </joint>
+    <joint name="right_friction_joint">
+      <command_interface name="velocity"/>
+      <command_interface name="effort"/>
+      <state_interface name="position"/>
+      <state_interface name="velocity"/>
+    </joint>
+    <joint name="bullet_feeder_joint">
+      <command_interface name="velocity"/>
+      <command_interface name="effort"/>
+      <state_interface name="position"/>
+      <state_interface name="velocity"/>
+    </joint>
+  </ros2_control>
+  <ros2_control name="CommandGz" type="system">
+    <hardware>
+      <plugin>$(arg command_hardware_plugin)</plugin>
+    </hardware>
+    <gpio name="command/chassis/linear/x">
+      <command_interface name="velocity"/>
+      <state_interface name="velocity"/>
+    </gpio>
+    <gpio name="command/chassis/linear/y">
+      <command_interface name="velocity"/>
+      <state_interface name="velocity"/>
+    </gpio>
+    <gpio name="command/chassis/angular/z">
+      <command_interface name="velocity"/>
+      <state_interface name="velocity"/>
+    </gpio>
+    <gpio name="command/chassis">
+      <command_interface name="mode"/>
+      <state_interface name="mode"/>
+    </gpio>
+    <gpio name="command/gimbal/yaw">
+      <command_interface name="velocity"/>
+      <state_interface name="velocity"/>
+    </gpio>
+    <gpio name="command/gimbal/pitch">
+      <command_interface name="velocity"/>
+      <state_interface name="velocity"/>
+    </gpio>
+    <gpio name="command/gimbal">
+      <command_interface name="enabled"/>
+      <state_interface name="enabled"/>
+    </gpio>
+    <gpio name="command/shooter">
+      <command_interface name="mode"/>
+      <command_interface name="sequence"/>
+      <state_interface name="mode"/>
+      <state_interface name="sequence"/>
+    </gpio>
   </ros2_control>
   <gazebo>
