Commit message: feat(sim): add omni infantry gazebo bringup

File: rmgo_ws/src/rmgo_description/urdf/omni_infantry_gz.urdf.xacro (robot description, xacro)
@@ -3,9 +3,22 @@
   <xacro:arg name="hardware_plugin" default="gz_ros2_control/GazeboSimSystem"/>
   <xacro:arg name="controllers_file" default="$(find rmgo_description)/config/omni_infantry_controllers.yaml"/>
+  <xacro:arg name="debug_visuals" default="false"/>
   <xacro:property name="wheel_distance_x" value="0.31794"/>
   <xacro:property name="wheel_distance_y" value="0.31794"/>
+  <xacro:property name="wheel_radius" value="0.07"/>
+  <xacro:property name="roller_radius" value="0.012"/>
+  <xacro:property name="roller_ring_radius" value="${wheel_radius - roller_radius}"/>
   <xacro:property name="gimbal_center_height" value="0.32059"/>
   <material name="white">
     <color rgba="1 1 1 1"/>
+  </material>
+  <material name="black">
+    <color rgba="0.02 0.02 0.02 1"/>
+  </material>
+  <material name="chassis_gray">
+    <color rgba="0.36 0.38 0.36 1"/>
+  </material>
+  <material name="gimbal_orange">
+    <color rgba="0.92 0.42 0.12 1"/>
   </material>
   <xacro:macro name="box_inertial" params="mass x y z">
@@ -33,4 +46,16 @@
     </inertial>
   </xacro:macro>
+  <xacro:macro name="sphere_inertial" params="mass radius">
+    <inertial>
+      <mass value="${mass}"/>
+      <inertia
+        ixx="${2.0 * mass * radius * radius / 5.0}"
+        ixy="0.0"
+        ixz="0.0"
+        iyy="${2.0 * mass * radius * radius / 5.0}"
+        iyz="0.0"
+        izz="${2.0 * mass * radius * radius / 5.0}"/>
+    </inertial>
+  </xacro:macro>
   <xacro:macro name="tiny_inertial" params="mass">
     <inertial>
@@ -45,4 +70,32 @@
       </geometry>
     </collision>
+  </xacro:macro>
+  <xacro:macro name="box_visual" params="name x y z material origin_xyz:='0 0 0'">
+    <visual name="${name}">
+      <origin xyz="${origin_xyz}"/>
+      <geometry>
+        <box size="${x} ${y} ${z}"/>
+      </geometry>
+      <material name="${material}"/>
+    </visual>
+  </xacro:macro>
+  <xacro:macro name="debug_box_visual" params="name x y z material origin_xyz:='0 0 0'">
+    <xacro:if value="$(arg debug_visuals)">
+      <xacro:box_visual name="${name}" x="${x}" y="${y}" z="${z}" material="${material}" origin_xyz="${origin_xyz}"/>
+    </xacro:if>
+  </xacro:macro>
+  <xacro:macro name="x_cylinder_visual" params="name radius length material">
+    <visual name="${name}">
+      <origin rpy="0 ${pi/2} 0"/>
+      <geometry>
+        <cylinder radius="${radius}" length="${length}"/>
+      </geometry>
+      <material name="${material}"/>
+    </visual>
+  </xacro:macro>
+  <xacro:macro name="debug_x_cylinder_visual" params="name radius length material">
+    <xacro:if value="$(arg debug_visuals)">
+      <xacro:x_cylinder_visual name="${name}" radius="${radius}" length="${length}" material="${material}"/>
+    </xacro:if>
   </xacro:macro>
   <xacro:macro name="stl_visual" params="filename">
@@ -57,38 +110,91 @@
     <xacro:box_inertial mass="10.0" x="0.45" y="0.45" z="0.12"/>
     <xacro:stl_visual filename="base_link.stl"/>
-    <xacro:box_collision x="0.45" y="0.45" z="0.12"/>
-  </link>
-  <xacro:macro name="generate_wheel" params="name rpy xyz">
-    <link name="${name}_wheel_link">
-      <xacro:x_cylinder_inertial mass="0.5" radius="0.07" length="0.05"/>
-      <xacro:stl_visual filename="wheel_link.stl"/>
+    <xacro:debug_box_visual name="base_debug_visual" x="0.45" y="0.45" z="0.12" material="chassis_gray" origin_xyz="0 0 0.11"/>
+    <collision>
+      <origin xyz="0 0 0.11"/>
+      <geometry>
+        <box size="0.45 0.45 0.12"/>
+      </geometry>
+    </collision>
+  </link>
+  <gazebo reference="base_link">
+    <mu1 value="1.0"/>
+    <mu2 value="1.0"/>
+    <kp value="1000000.0"/>
+    <kd value="100.0"/>
+  </gazebo>
+  <xacro:macro name="generate_roller" params="wheel index theta">
+    <link name="${wheel}_roller_${index}_link">
+      <xacro:sphere_inertial mass="0.006" radius="${roller_radius}"/>
       <collision>
-        <origin rpy="0 ${pi/2} 0"/>
         <geometry>
-          <cylinder radius="0.07" length="0.05"/>
+          <sphere radius="${roller_radius}"/>
         </geometry>
       </collision>
+      <visual>
+        <geometry>
+          <sphere radius="${roller_radius}"/>
+        </geometry>
+        <material name="black"/>
+      </visual>
+    </link>
+    <joint name="${wheel}_roller_${index}_joint" type="continuous">
+      <origin xyz="0 ${roller_ring_radius * cos(theta)} ${roller_ring_radius * sin(theta)}"/>
+      <axis xyz="0 ${-sin(theta)} ${cos(theta)}"/>
+      <dynamics damping="0.0" friction="0.001"/>
+      <parent link="${wheel}_wheel_link"/>
+      <child link="${wheel}_roller_${index}_link"/>
+    </joint>
+    <gazebo reference="${wheel}_roller_${index}_link">
+      <mu1 value="2000.0"/>
+      <mu2 value="2000.0"/>
+      <kp value="1000000.0"/>
+      <kd value="100.0"/>
+      <material>Gazebo/Black</material>
+    </gazebo>
+  </xacro:macro>
+  <xacro:macro name="generate_roller_ring" params="wheel">
+    <xacro:generate_roller wheel="${wheel}" index="0" theta="${0*pi/6}"/>
+    <xacro:generate_roller wheel="${wheel}" index="1" theta="${1*pi/6}"/>
+    <xacro:generate_roller wheel="${wheel}" index="2" theta="${2*pi/6}"/>
+    <xacro:generate_roller wheel="${wheel}" index="3" theta="${3*pi/6}"/>
+    <xacro:generate_roller wheel="${wheel}" index="4" theta="${4*pi/6}"/>
+    <xacro:generate_roller wheel="${wheel}" index="5" theta="${5*pi/6}"/>
+    <xacro:generate_roller wheel="${wheel}" index="6" theta="${6*pi/6}"/>
+    <xacro:generate_roller wheel="${wheel}" index="7" theta="${7*pi/6}"/>
+    <xacro:generate_roller wheel="${wheel}" index="8" theta="${8*pi/6}"/>
+    <xacro:generate_roller wheel="${wheel}" index="9" theta="${9*pi/6}"/>
+    <xacro:generate_roller wheel="${wheel}" index="10" theta="${10*pi/6}"/>
+    <xacro:generate_roller wheel="${wheel}" index="11" theta="${11*pi/6}"/>
+  </xacro:macro>
+  <xacro:macro name="generate_omni_wheel" params="name rpy xyz">
+    <link name="${name}_wheel_link">
+      <xacro:x_cylinder_inertial mass="0.45" radius="${wheel_radius}" length="0.05"/>
+      <xacro:stl_visual filename="wheel_link.stl"/>
+      <xacro:debug_x_cylinder_visual name="${name}_wheel_debug_visual" radius="${wheel_radius}" length="0.05" material="black"/>
     </link>
     <joint name="${name}_wheel_joint" type="continuous">
       <axis xyz="1 0 0"/>
       <limit effort="20.0" velocity="40.0"/>
+      <dynamics damping="0.0" friction="0.02"/>
       <parent link="base_link"/>
       <child link="${name}_wheel_link"/>
       <origin rpy="${rpy}" xyz="${xyz}"/>
     </joint>
-  </xacro:macro>
-  <xacro:generate_wheel
+    <xacro:generate_roller_ring wheel="${name}"/>
+  </xacro:macro>
+  <xacro:generate_omni_wheel
     name="left_front"
     rpy="0 0 ${pi/4}"
     xyz="${wheel_distance_x/2} ${wheel_distance_y/2} 0"/>
-  <xacro:generate_wheel
+  <xacro:generate_omni_wheel
     name="left_back"
     rpy="0 0 ${3*pi/4}"
     xyz="-${wheel_distance_x/2} ${wheel_distance_y/2} 0"/>
-  <xacro:generate_wheel
+  <xacro:generate_omni_wheel
     name="right_back"
     rpy="0 0 -${3*pi/4}"
     xyz="-${wheel_distance_x/2} -${wheel_distance_y/2} 0"/>
-  <xacro:generate_wheel
+  <xacro:generate_omni_wheel
     name="right_front"
     rpy="0 0 -${pi/4}"
@@ -97,4 +203,5 @@
     <xacro:box_inertial mass="2.0" x="0.18" y="0.18" z="0.12"/>
     <xacro:stl_visual filename="yaw_link.stl"/>
+    <xacro:debug_box_visual name="yaw_debug_visual" x="0.18" y="0.18" z="0.12" material="gimbal_orange"/>
     <xacro:box_collision x="0.18" y="0.18" z="0.12"/>
   </link>
@@ -109,4 +216,5 @@
     <xacro:box_inertial mass="1.0" x="0.20" y="0.12" z="0.12"/>
     <xacro:stl_visual filename="pitch_link.stl"/>
+    <xacro:debug_box_visual name="pitch_debug_visual" x="0.20" y="0.12" z="0.12" material="gimbal_orange"/>
     <xacro:box_collision x="0.20" y="0.12" z="0.12"/>
   </link>

Commit message: feat(sim): model gimbal actuator dynamics

File: rmgo_ws/src/rmgo_description/urdf/omni_infantry_gz.urdf.xacro (robot description, xacro)
@@ -208,5 +208,6 @@
   <joint name="yaw_joint" type="continuous">
     <axis xyz="0 0 1"/>
-    <limit effort="10.0" velocity="6.0"/>
+    <limit effort="25.0" velocity="12.0"/>
+    <dynamics damping="0.08" friction="0.02"/>
     <parent link="base_link"/>
     <child link="yaw_link"/>
@@ -221,5 +222,6 @@
   <joint name="pitch_joint" type="continuous">
     <axis xyz="0 1 0"/>
-    <limit effort="10.0" velocity="6.0"/>
+    <limit effort="6.0" velocity="4.0"/>
+    <dynamics damping="0.2" friction="0.04"/>
     <parent link="yaw_link"/>
     <child link="pitch_link"/>
@@ -274,10 +276,24 @@
     </joint>
     <joint name="yaw_joint">
-      <command_interface name="position"/>
+      <command_interface name="position">
+        <param name="sim_servo_kp">36.0</param>
+        <param name="sim_servo_kd">5.0</param>
+        <param name="sim_servo_max_effort">25.0</param>
+        <param name="sim_servo_max_velocity">16.0</param>
+        <param name="sim_servo_deadband">0.0001</param>
+        <param name="sim_servo_velocity_feedforward">1.0</param>
+      </command_interface>
       <state_interface name="position"/>
       <state_interface name="velocity"/>
     </joint>
     <joint name="pitch_joint">
-      <command_interface name="position"/>
+      <command_interface name="position">
+        <param name="sim_servo_kp">6.0</param>
+        <param name="sim_servo_kd">0.8</param>
+        <param name="sim_servo_max_effort">2.0</param>
+        <param name="sim_servo_max_velocity">2.0</param>
+        <param name="sim_servo_deadband">0.0005</param>
+        <param name="sim_servo_velocity_feedforward">0.2</param>
+      </command_interface>
       <state_interface name="position"/>
       <state_interface name="velocity"/>

Commit message: fix: stabilize gazebo shooter simulation

File: rmgo_ws/src/rmgo_description/urdf/omni_infantry_gz.urdf.xacro (robot description, xacro)
@@ -235,5 +235,5 @@
     <axis xyz="1 0 0"/>
     <limit effort="2.0" velocity="800.0"/>
-    <dynamics damping="0.0" friction="0.001"/>
+    <dynamics damping="0.003" friction="0.001"/>
     <parent link="pitch_link"/>
     <child link="left_friction_link"/>
@@ -247,5 +247,5 @@
     <axis xyz="1 0 0"/>
     <limit effort="2.0" velocity="800.0"/>
-    <dynamics damping="0.0" friction="0.001"/>
+    <dynamics damping="0.003" friction="0.001"/>
     <parent link="pitch_link"/>
     <child link="right_friction_link"/>
@@ -259,5 +259,5 @@
     <axis xyz="1 0 0"/>
     <limit effort="4.0" velocity="60.0"/>
-    <dynamics damping="0.01" friction="0.002"/>
+    <dynamics damping="0.005" friction="0.002"/>
     <parent link="pitch_link"/>
     <child link="bullet_feeder_link"/>
